File: AN001-Appnote-brd/SomTest1.sch (EAGLE design)
At the start: 43 parts, among them J1 SPARK_M.2EKEY, U1 MAX17043, U2 BQ24195, U3 XCL223

Commit message: added ricks basic som design as a base
Changed lines of the file:
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@@
 <?xml version="1.0" encoding="utf-8"?>
 <!DOCTYPE eagle SYSTEM "eagle.dtd">
-<eagle version="9.6.2">
+<eagle version="9.4.0">
 <drawing>
 <settings>
-<setting alwaysvectorfont="no"/>
+<setting alwaysvectorfont="yes"/>
 <setting verticaltext="up"/>
 </settings>
@@
 </plain>
 <instances>
-</instances>
-<busses>
-</busses>
-<nets>
-</nets>
-</sheet>
-<sheet>
-<plain>
-</plain>
-<instances>
 <instance part="R1" gate="G$1" x="124.46" y="58.42" smashed="yes" rot="R90">
 <attribute name="NAME" x="122.9614" y="54.61" size="1.778" layer="95" rot="R90"/>
@@
 </sheet>
 </sheets>
+<errors>
+</errors>
 </schematic>
 </drawing>
