File: m2_feather_interposer/m2_feather_interposer.sch (EAGLE design)
At the start: 43 parts, among them J1 SPARK_M.2EKEY, U1 MAX17043, U2 BQ24195, U3 XCL223

Commit message: added a whole bunch of stuff, board layout, draft key component placements, added connectors, added components from the boron that were missing.
Parts:
- removed C13: 4.7uF, rickk2:CAP-4.7UF-0603
- removed C14: 10uF, rickk2:CAP-10UF-0603
- removed CN1: (no value), rickk2:JST_2PIN-THM
- removed JP1: M02PTH, rickk2:M02PTH
- removed S1, S2: SWITCH-MOM-4.5, rickk2:SWITCH-MOM-4.5
- removed U3: XCL223, rickk2:REG-XCL223
- added C15, C16, C17: 47pF, m2_feather_interposer:PARTICLE_C-USC0201_B
- added C50: 100nF, m2_feather_interposer:PARTICLE_C-USC0201_B
- added J3: (no value), SparkFun-Connectors:CONN_02
- added MS1: MICROBUILDER_FEATHERWINGSMT_BTM_FEATHER, m2_feather_interposer:MICROBUILDER_FEATHERWINGSMT_BTM_FEATHER
- added NFC: UFL, m2_feather_interposer:PARTICLE_IPEX-20279-001E
- added R37, R38: ESD NC, m2_feather_interposer:REDBEAR_RES0402S
- added S5, S6: B3U-3000P-B, m2_feather_interposer:B3U-3000P-B
- added U$4: M2_FEATHER_INTERPOSER_PARTICLE_SIM-NANO-4FF, m2_feather_interposer:M2_FEATHER_INTERPOSER_PARTICLE_SIM-NANO-4FF
- added U4: PARTICLE_XC9258A33EER-G, m2_feather_interposer:PARTICLE_XC9258A33EER-G
- added U5: PARTICLE_XC8107SOT25, m2_feather_interposer:PARTICLE_XC8107SOT25
- C1: device rickk2:CAP-0.01UF-0603 -> m2_feather_interposer:RICKK2_CAP-0.01UF-0603
- C10, C4, C5, C6, C7, C9: device rickk2:CAP-10UF-0603 -> m2_feather_interposer:RICKK2_CAP-10UF-0603
- C11: device rickk2:CAP-0.001UF-0603 -> m2_feather_interposer:RICKK2_CAP-0.001UF-0603
- C12: device rickk2:CAP-0.047UF-0603 -> m2_feather_interposer:RICKK2_CAP-0.047UF-0603
- C8: device rickk2:CAP-4.7UF-0603 -> m2_feather_interposer:RICKK2_CAP-4.7UF-0603
- D1: device rickk2:LED-RED -> m2_feather_interposer:RICKK2_LED-RED
- D2: device rickk2:DIODE-RS1JFP -> m2_feather_interposer:RICKK2_DIODE-RS1JFP
- J1: value SPARK_M.2EKEY -> RICKK2_SPARK_M.2EKEY; device rickk2:SPARK_M.2EKEY -> m2_feather_interposer:RICKK2_SPARK_M.2EKEY
- L1: device rickk2:INDUCTOR-2.2UH -> m2_feather_interposer:RICKK2_INDUCTOR-2.2UH
- LED1: value LED-RGB-CREE-SMD -> RICKK2_LED-RGB-CREE-SMD; device rickk2:LED-RGB-CREE-SMD -> m2_feather_interposer:RICKK2_LED-RGB-CREE-SMD
- R1, R10, R11, R15, R9: device rickk2:RES-10K-06030603 -> m2_feather_interposer:RICKK2_RES-10K-06030603
- R12, R2, R3, R4, R6: device rickk2:RES-1K-0603 -> m2_feather_interposer:RICKK2_RES-1K-0603
- R14: device rickk2:RES-5.6K-0603 -> m2_feather_interposer:RICKK2_RES-5.6K-0603
- R5: device rickk2:RES-150-0603 -> m2_feather_interposer:RICKK2_RES-150-0603
- R7, R8: device rickk2:RES-4.7K-0603 -> m2_feather_interposer:RICKK2_RES-4.7K-0603
- U$1: value M2-STANDOFF -> RICKK2_M2-STANDOFF; device rickk2:M2-STANDOFF -> m2_feather_interposer:RICKK2_M2-STANDOFF
- U$3: value USB-MICRO-B-SOCKET-AMPHENOL -> RICKK2_USB-MICRO-B-SOCKET-AMPHENOL; device rickk2:USB-MICRO-B-SOCKET-AMPHENOL -> m2_feather_interposer:RICKK2_USB-MICRO-B-SOCKET-AMPHENOL
- U1: device rickk2:MAX17043 -> m2_feather_interposer:RICKK2_MAX17043
- U2: device rickk2:BQ24195 -> m2_feather_interposer:RICKK2_BQ24195
Connections:
- removed net L2: U3.L2, U3.LX
- new net A0: J1.A0, MS1.GPIOA0
- new net A1: J1.A1, MS1.GPIOA1
- new net A2: J1.A2, MS1.GPIOA2
- new net A3: J1.A3, MS1.GPIOA3
- new net A4: J1.A4, MS1.GPIOA4
- new net A5: J1.A5, MS1.GPIOA5
- new net D2: MS1.GPIO5
- new net D3: MS1.GPIO6
- new net D4: MS1.GPIO9
- new net D5: MS1.GPIO10
- new net D6: MS1.GPIO11
- new net D7: MS1.GPIO12
- new net D8: MS1.GPIO13
- new net MISO: J1.MISO, MS1.GPIOMISO
- new net MOSI: J1.MOSI, MS1.GPIOMOSI
- new net NANO_CLK: C16.1
- new net NANO_DATA: C17.1
- new net NANO_RST: C15.1
- new net NANO_VSIM: C50.1
- new net NFC1: NFC.GND@1, R37.1
- new net NFC2: NFC.1, R38.2
- new net RX: J1.RX, MS1.GPIORX
- new net SCK: J1.SCK, MS1.GPIOSCK
- new net SYS_PWR_EN: MS1.EN, U5.CE
- new net TX: J1.TX, MS1.GPIOTX
- net /MODE: now also MS1.AREF, S5.2; no longer S1.3
- net /RESET: now also MS1.!RESET, S6.2; no longer S2.3
- net 3V3: now also MS1.3V; no longer C14.1, U3.L1, U3.VOUT
- net 3V7: now also U4.VIN; no longer C13.1, U3.CE, U3.VIN
- net BAT: now also J3.1, MS1.VBAT; no longer CN1.2
- net GND: now also C15.2, C16.2, C17.2, C50.2, J3.2, MS1.GND, R37.2, R38.1, S5.1, S6.1, U4.VSS@2, U4.VSS@5, U5.VSS; no longer C13.2, C14.2, CN1.1, JP1.2, S1.2, S2.2, U3.AGND, U3.PGND
- net SCL: now also MS1.GPIOSCL
- net SDA: now also MS1.GPIOSDA
- net VBUS: now also MS1.USB; no longer JP1.1

Commit message: all components added and key component placement done, driving through layout draft
Parts:
- removed U1: MAX17043, m2_feather_interposer:RICKK2_MAX17043
- removed U4: PARTICLE_XC9258A33EER-G, m2_feather_interposer:PARTICLE_XC9258A33EER-G
- removed U5: PARTICLE_XC8107SOT25, m2_feather_interposer:PARTICLE_XC8107SOT25
- added C18, C19: 10uF/10V, rcl:C-USC0603K
- added C20: 100nF, rcl:C-USC0603K
- added C21: 100nF, Particle:C-USC0201_B
- added D3: P1.03, SparkFun-LED:LED-RED0603
- added L2: 4.7uH, Particle:INDUCTOR-SPARKFUNVLS3012ET-4R7M
- added R11_, R16: 10K, adafruit:R-US_R0402
- added R13_: 332, adafruit:R-US_R0402
- added R17: 100k, adafruit:R-US_R0402
- added R19: 1K, Particle:R-US_R0201_B
- added U3: MAX1704X, SparkFun-IC-Power:MAX1704X
- added U6: XC9258A33EER-G, Particle:XC9258A33EER-G
- added U7: XC8107SOT25, Particle:XC8107SOT25
- C1: device m2_feather_interposer:RICKK2_CAP-0.01UF-0603 -> adafruit:C-USC0402
- C11: device m2_feather_interposer:RICKK2_CAP-0.001UF-0603 -> adafruit:C-USC0402
- C12: device m2_feather_interposer:RICKK2_CAP-0.047UF-0603 -> adafruit:C-USC0402
- C3: device rickk2:CAP-1UF-0603.DEV -> adafruit:C-USC0402
- R1, R10, R15, R9: device m2_feather_interposer:RICKK2_RES-10K-06030603 -> adafruit:R-US_R0402
- R11: value 10K -> 0; device m2_feather_interposer:RICKK2_RES-10K-06030603 -> adafruit:R-US_R0402
- R12: device m2_feather_interposer:RICKK2_RES-1K-0603 -> adafruit:R-US_R0402
- R13: value 332 -> 0; device rickk2:RES-332-0603.DEV -> adafruit:R-US_R0402
- R14: device m2_feather_interposer:RICKK2_RES-5.6K-0603 -> adafruit:R-US_R0402
- R2, R3, R4: value 1K -> 1k; device m2_feather_interposer:RICKK2_RES-1K-0603 -> adafruit:R-US_R0402
- R5: device m2_feather_interposer:RICKK2_RES-150-0603 -> adafruit:R-US_R0402
- R6: value 1K -> 4.7K; device m2_feather_interposer:RICKK2_RES-1K-0603 -> adafruit:R-US_R0402
- R7, R8: device m2_feather_interposer:RICKK2_RES-4.7K-0603 -> adafruit:R-US_R0402
Connections:
- new net N$23: R16.2, U6.CE
- new net N$24: D3.C, R19.2
- new net N$25: L2.1, U6.LX
- new net N$4: R11.1, U$3.D+
- new net N$8: R13.1, U$3.D-
- new net PMIC_VSYS: C10.1, C11.1, C9.1, L1.P$2, R12.2, R17.2, U2.SYS@15, U2.SYS@16, U7.VIN
- new net USB_D_N: J1.USB-D-, R13.2
- new net USB_D_P: J1.USB-D+, R11.2
- net 3V3: now also C19.1, C21.1, L2.2, U6.VOUT
- net 3V7: now also C18.1, C20.1, R16.1, U6.VIN, U7.VOUT; no longer C10.1, C11.1, C9.1, L1.P$2, R12.2, U2.SYS@15, U2.SYS@16, U4.VIN
- net BATINT: now also U3.ALT; no longer U1./ALRT
- net BQCE: now also R11_.2; no longer R11.2
- net D2: now also J1.D2
- net D3: now also J1.D3
- net D4: now also J1.D4
- net D5: now also J1.D5
- net D6: now also J1.D6
- net D7: now also D3.A, J1.D7
- net D8: now also J1.CS
- net GND: now also C18.2, C19.2, C20.2, C21.2, R11_.1, R13_.1, R19.1, U$4.GND, U3.CTG, U3.GND@4, U3.GND@EP, U3.QST, U6.VSS@2, U6.VSS@5, U7.VSS; no longer R11.1, R13.1, U1.CTG, U1.GND, U1.QSTRT, U4.VSS@2, U4.VSS@5, U5.VSS
- net ILIM: now also R13_.2; no longer R13.2
- net N$3: now also U3.CELL; no longer U1.CELL
- net N$5: now also U3.VDD; no longer U1.VDD
- net NANO_CLK: now also J1.SOM7, U$4.CLK
- net NANO_DATA: now also J1.SOM8, U$4.I/O
- net NANO_RST: now also J1.SOM6, U$4.RST
- net NANO_VSIM: now also J1.SOM5, U$4.VCC
- net NFC1: now also J1.SOM3
- net NFC2: now also J1.SOM4
- net SCL: now also U3.SCL; no longer U1.SCL
- net SDA: now also U3.SDA; no longer U1.SDA
- net SYS_PWR_EN: now also R17.1, U7.CE; no longer U5.CE
- net USB-D+: no longer J1.USB-D+, U$3.D+
- net USB-D-: no longer J1.USB-D-, U$3.D-
Other:
- note added: "3.3V REGULATOR"
- note added: "OUTPUT IS 3.7V"
- note added: "POWER SWITCH"
- note added: "high precision 1k"
- moved on the sheet: C15, C16, C17, C50, LED1, NFC, R11, R13, R2, R3, R37, R38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
