File: m2_feather_interposer/m2_feather_interposer.sch (EAGLE design)
At the start: 62 parts, among them J1 RICKK2_SPARK_M.2EKEY, U2 BQ24195, U3 MAX1704X, U6 XC9258A33EER-G, U7 XC8107SOT25

Commit message: added draft bom
Parts:
- removed C13: 10uF, m2_feather_interposer:RICKK2_CAP-10UF-0603
- removed S5, S6: B3U-3000P-B, m2_feather_interposer:B3U-3000P-B
- added S1, S2: B3U-3000P, m2_feather_interposer:B3U-3000P
- D3: value P1.03 -> RED
- R19: value 1K -> 1k; device Particle:R-US_R0201_B -> adafruit:R-US_R0402
- renumbered R13_ to R131
Connections:
- net /MODE: now also S1.2; no longer S5.2
- net /RESET: now also S2.2; no longer S6.2
- net GND: now also R19.2, S1.1, S2.1; no longer C13.2, R19.1, S5.1, S6.1
- net N$24: now also R19.1; no longer R19.2
- net PMID: no longer C13.1
Changed lines of the file:
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@@
 <setting verticaltext="up"/>
 </settings>
-<grid distance="0.05" unitdist="inch" unit="inch" style="lines" multiple="1" display="no" altdistance="0.01" altunitdist="inch" altunit="inch"/>
+<grid distance="0.1" unitdist="inch" unit="inch" style="lines" multiple="1" display="no" altdistance="0.01" altunitdist="inch" altunit="inch"/>
 <layers>
 <layer number="1" name="Top" color="4" fill="1" visible="no" active="no"/>
@@
 <part name="GND60" library="m2_feather_interposer" deviceset="REDBEAR-DUO_GND" device=""/>
 <part name="GND62" library="m2_feather_interposer" deviceset="REDBEAR-DUO_GND" device=""/>
-<part name="S5" library="m2_feather_interposer" deviceset="B3U-3000P-B" device=""/>
-<part name="S6" library="m2_feather_interposer" deviceset="B3U-3000P-B" device=""/>
 <part name="J3" library="SparkFun-Connectors" library_urn="urn:adsk.eagle:library:513" deviceset="CONN_02" device="" package3d_urn="urn:adsk.eagle:package:38039/1"/>
 <part name="GND6" library="m2_feather_interposer" deviceset="RICKK2_GND" device=""/>
@@
 <part name="R9" library="adafruit" library_urn="urn:adsk.eagle:library:420" deviceset="R-US_" device="R0402" package3d_urn="urn:adsk.eagle:package:6240564/1" value="10K"/>
 <part name="R10" library="adafruit" library_urn="urn:adsk.eagle:library:420" deviceset="R-US_" device="R0402" package3d_urn="urn:adsk.eagle:package:6240564/1" value="10K"/>
-<part name="R13_" library="adafruit" library_urn="urn:adsk.eagle:library:420" deviceset="R-US_" device="R0402" package3d_urn="urn:adsk.eagle:package:6240564/1" value="332"/>
+<part name="R131" library="adafruit" library_urn="urn:adsk.eagle:library:420" deviceset="R-US_" device="R0402" package3d_urn="urn:adsk.eagle:package:6240564/1" value="332"/>
 <part name="R11_" library="adafruit" library_urn="urn:adsk.eagle:library:420" deviceset="R-US_" device="R0402" package3d_urn="urn:adsk.eagle:package:6240564/1" value="10K"/>
 <part name="R15" library="adafruit" library_urn="urn:adsk.eagle:library:420" deviceset="R-US_" device="R0402" package3d_urn="urn:adsk.eagle:package:6240564/1" value="10K"/>
@@
 <part name="C11" library="adafruit" library_urn="urn:adsk.eagle:library:420" deviceset="C-US" device="C0402" package3d_urn="urn:adsk.eagle:package:6240340/1" value="0.001uF"/>
 <part name="C12" library="adafruit" library_urn="urn:adsk.eagle:library:420" deviceset="C-US" device="C0402" package3d_urn="urn:adsk.eagle:package:6240340/1" value="0.047uF"/>
-<part name="D3" library="SparkFun-LED" deviceset="LED-RED" device="0603" value="P1.03"/>
-<part name="R19" library="Particle" deviceset="R-US_" device="R0201_B" value="1K"/>
+<part name="D3" library="SparkFun-LED" library_urn="urn:adsk.eagle:library:529" deviceset="LED-RED" device="0603" package3d_urn="urn:adsk.eagle:package:39354/1" value="RED"/>
 <part name="GND74" library="supply1" deviceset="GND" device=""/>
 <part name="U3" library="SparkFun-IC-Power" library_urn="urn:adsk.eagle:library:526" deviceset="MAX1704X" device="" package3d_urn="urn:adsk.eagle:package:39055/1"/>
 <part name="R11" library="adafruit" library_urn="urn:adsk.eagle:library:420" deviceset="R-US_" device="R0402" package3d_urn="urn:adsk.eagle:package:6240564/1" value="0"/>
 <part name="R13" library="adafruit" library_urn="urn:adsk.eagle:library:420" deviceset="R-US_" device="R0402" package3d_urn="urn:adsk.eagle:package:6240564/1" value="0"/>
-<part name="C13" library="m2_feather_interposer" deviceset="RICKK2_CAP-10UF-0603" device="" value="10uF"/>
+<part name="S1" library="m2_feather_interposer" deviceset="B3U-3000P" device=""/>
+<part name="S2" library="m2_feather_interposer" deviceset="B3U-3000P" device=""/>
+<part name="R19" library="adafruit" library_urn="urn:adsk.eagle:library:420" deviceset="R-US_" device="R0402" package3d_urn="urn:adsk.eagle:package:6240564/1" value="1k"/>
 </parts>
 <sheets>
@@
 <attribute name="VALUE" x="236.22" y="198.12" size="1.778" layer="96" rot="R180"/>
 </instance>
-<instance part="S5" gate="G$1" x="144.78" y="48.26" smashed="yes">
-<attribute name="NAME" x="152.4104" y="45.71653125" size="2.54346875" layer="95"/>
-<attribute name="VALUE" x="152.40033125" y="40.63966875" size="2.540109375" layer="96"/>
-</instance>
-<instance part="S6" gate="G$1" x="139.7" y="22.86" smashed="yes">
-<attribute name="NAME" x="147.3304" y="20.31653125" size="2.54346875" layer="95"/>
-<attribute name="VALUE" x="147.32033125" y="15.23966875" size="2.540109375" layer="96"/>
-</instance>
 <instance part="J3" gate="G$1" x="152.4" y="162.56" smashed="yes" rot="R180">
 <attribute name="VALUE" x="154.94" y="167.386" size="1.778" layer="96" font="vector" rot="R180"/>
@@
 <attribute name="VALUE" x="28.702" y="151.13" size="1.778" layer="96" rot="R90"/>
 </instance>
-<instance part="R13_" gate="G$1" x="17.78" y="129.54" smashed="yes" rot="R90">
+<instance part="R131" gate="G$1" x="17.78" y="129.54" smashed="yes" rot="R90">
 <attribute name="NAME" x="16.2814" y="125.73" size="1.778" layer="95" rot="R90"/>
 <attribute name="VALUE" x="21.082" y="125.73" size="1.778" layer="96" rot="R90"/>
@@
 <attribute name="VALUE" x="271.272" y="14.605" size="1.778" layer="96" font="vector" rot="R180" align="top-left"/>
 </instance>
-<instance part="R19" gate="R1" x="279.4" y="12.7" smashed="yes" rot="R180">
-<attribute name="NAME" x="283.21" y="11.2014" size="1.778" layer="95" rot="R180"/>
-<attribute name="VALUE" x="283.21" y="16.002" size="1.778" layer="96" rot="R180"/>
-</instance>
 <instance part="GND74" gate="1" x="284.48" y="5.08" smashed="yes">
 <attribute name="VALUE" x="281.94" y="2.54" size="1.778" layer="96"/>
@@
 <attribute name="VALUE" x="20.32" y="74.168" size="1.778" layer="96"/>
 </instance>
-<instance part="C13" gate="G$1" x="13.97" y="172.72" smashed="yes">
-<attribute name="NAME" x="15.494" y="175.641" size="1.778" layer="95"/>
-<attribute name="VALUE" x="15.494" y="170.561" size="1.778" layer="96"/>
+<instance part="S1" gate="G$1" x="144.78" y="48.26" smashed="yes">
+<attribute name="NAME" x="152.4104" y="45.71653125" size="2.54346875" layer="95"/>
+<attribute name="VALUE" x="152.40033125" y="40.63966875" size="2.540109375" layer="96"/>
+</instance>
+<instance part="S2" gate="G$1" x="139.7" y="22.86" smashed="yes">
+<attribute name="NAME" x="147.3304" y="20.31653125" size="2.54346875" layer="95"/>
+<attribute name="VALUE" x="147.32033125" y="15.23966875" size="2.540109375" layer="96"/>
+</instance>
+<instance part="R19" gate="G$1" x="279.4" y="12.7" smashed="yes">
+<attribute name="NAME" x="275.59" y="14.1986" size="1.778" layer="95"/>
+<attribute name="VALUE" x="275.59" y="9.398" size="1.778" layer="96"/>
 </instance>
 </instances>
@@
 <wire x1="162.56" y1="25.4" x2="162.56" y2="17.78" width="0.1524" layer="91"/>
 <wire x1="152.4" y1="25.4" x2="162.56" y2="25.4" width="0.1524" layer="91"/>
-<pinref part="S6" gate="G$1" pin="1"/>
-<pinref part="S5" gate="G$1" pin="1"/>
 <wire x1="157.48" y1="50.8" x2="162.56" y2="50.8" width="0.1524" layer="91"/>
 <wire x1="162.56" y1="50.8" x2="162.56" y2="25.4" width="0.1524" layer="91"/>
 <junction x="162.56" y="25.4"/>
+<pinref part="S1" gate="G$1" pin="1"/>
+<pinref part="S2" gate="G$1" pin="1"/>
 </segment>
 <segment>
@@
 <junction x="-22.86" y="167.64"/>
 <label x="-31.75" y="167.64" size="1.778" layer="95"/>
-<pinref part="R13_" gate="G$1" pin="1"/>
+<pinref part="R131" gate="G$1" pin="1"/>
 <pinref part="R11_" gate="G$1" pin="1"/>
-<pinref part="C13" gate="G$1" pin="2"/>
-<wire x1="13.97" y1="170.18" x2="13.97" y2="167.64" width="0.1524" layer="91"/>
-<wire x1="13.97" y1="167.64" x2="7.62" y2="167.64" width="0.1524" layer="91"/>
 </segment>
 <segment>
@@
 </segment>
 <segment>
-<pinref part="R19" gate="R1" pin="1"/>
 <pinref part="GND74" gate="1" pin="GND"/>
 <wire x1="284.48" y1="7.62" x2="284.48" y2="12.7" width="0.1524" layer="91"/>
+<pinref part="R19" gate="G$1" pin="2"/>
 </segment>
 </net>
@@
 <label x="127" y="50.8" size="1.778" layer="95"/>
 <pinref part="J1" gate="G$1" pin="MODE"/>
-<pinref part="S5" gate="G$1" pin="2"/>
+<pinref part="S1" gate="G$1" pin="2"/>
 </segment>
 <segment>
@@
 <label x="127" y="33.02" size="1.778" layer="95"/>
 <pinref part="J1" gate="G$1" pin="RESET"/>
-<pinref part="S6" gate="G$1" pin="2"/>
 <wire x1="127" y1="25.4" x2="124.46" y2="25.4" width="0.1524" layer="91"/>
 <pinref part="R1" gate="G$1" pin="1"/>
+<pinref part="S2" gate="G$1" pin="2"/>
 </segment>
 <segment>
@@
 <wire x1="17.78" y1="175.26" x2="17.78" y2="134.62" width="0.1524" layer="91"/>
 <label x="17.78" y="134.62" size="1.778" layer="95" rot="R90"/>
-<pinref part="R13_" gate="G$1" pin="2"/>
+<pinref part="R131" gate="G$1" pin="2"/>
 </segment>
 </net>
@@
 <segment>
 <pinref part="U2" gate="G$1" pin="PMID"/>
-<wire x1="53.34" y1="180.34" x2="13.97" y2="180.34" width="0.1524" layer="91"/>
+<wire x1="53.34" y1="180.34" x2="7.62" y2="180.34" width="0.1524" layer="91"/>
 <pinref part="C4" gate="G$1" pin="1"/>
-<wire x1="13.97" y1="180.34" x2="7.62" y2="180.34" width="0.1524" layer="91"/>
 <wire x1="7.62" y1="180.34" x2="7.62" y2="177.8" width="0.1524" layer="91"/>
 <label x="12.7" y="180.34" size="1.778" layer="95"/>
-<pinref part="C13" gate="G$1" pin="1"/>
-<wire x1="13.97" y1="177.8" x2="13.97" y2="180.34" width="0.1524" layer="91"/>
-<junction x="13.97" y="180.34"/>
 </segment>
 </net>
@@
 <segment>
 <pinref part="D3" gate="G$1" pin="C"/>
-<pinref part="R19" gate="R1" pin="2"/>
 <wire x1="274.32" y1="12.7" x2="271.78" y2="12.7" width="0.1524" layer="91"/>
-</segment>
-</net>
+<pinref part="R19" gate="G$1" pin="1"/>
+</segment>
+</net>
